File: Xonik Waveshaper v1.0 w gp.brd (EAGLE design)
At the start: 63.5 x 28.3 mm, 94 parts, among them IC1 TL074D, IC2 TL074D, IC3 TL074D, IC4 TL072D, IC5 4013D, T1 2n3904

Commit message: New versions
Parts:
- C7: value 10pF -> 5pF
Other:
- board size 63.5 x 28.3 mm -> 63.5 x 28.2 mm
