File: Xonik Waveshaper v1.0 w gp.sch (EAGLE design)
At the start: 94 parts, among them IC1 TL074D, IC2 TL074D, IC3 TL074D, IC4 TL072D, IC5 4013D, T1 2n3904

Commit message: New versions
Parts:
- C7: value 10pF -> 5pF
Changed lines of the file:
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@@
 <part name="C5" library="resistor" deviceset="C-EU" device="C0805" value="100nF"/>
 <part name="C6" library="resistor" deviceset="C-EU" device="C0805" value="100nF"/>
-<part name="C7" library="resistor" deviceset="C-EU" device="C0805" value="10pF"/>
+<part name="C7" library="resistor" deviceset="C-EU" device="C0805" value="5pF"/>
 <part name="GND13" library="supply1" deviceset="GND" device=""/>
 <part name="55" library="resistor" deviceset="R-EU_" device="R0805" value="20k"/>
