File: Xonik Waveshaper v1.0.brd (EAGLE design)
At the start: 63.5 x 28.3 mm, 94 parts, among them IC1 TL074D, IC2 TL074D, IC3 TL074D, IC4 TL072D, IC5 4013D, T1 2n3904

Commit message: New versions
Parts:
- C7: value 10pF -> 5pF
Changed lines of the file:
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@@
 <layer number="24" name="bOrigins" color="15" fill="1" visible="yes" active="yes"/>
 <layer number="25" name="tNames" color="7" fill="1" visible="yes" active="yes"/>
-<layer number="26" name="bNames" color="7" fill="1" visible="no" active="yes"/>
+<layer number="26" name="bNames" color="7" fill="1" visible="yes" active="yes"/>
 <layer number="27" name="tValues" color="7" fill="1" visible="no" active="yes"/>
 <layer number="28" name="bValues" color="7" fill="1" visible="no" active="yes"/>
@@
 <wire x1="3.175" y1="28.245" x2="0" y2="25.07" width="0" layer="20"/>
 <wire x1="0" y1="25.07" x2="0" y2="0" width="0" layer="20"/>
-<circle x="5.08" y="14.605" radius="0.0635" width="0.4064" layer="25"/>
-<circle x="19.685" y="14.605" radius="0.0635" width="0.4064" layer="25"/>
-<circle x="37.465" y="14.605" radius="0.0635" width="0.4064" layer="25"/>
-<circle x="47.625" y="14.605" radius="0.0635" width="0.4064" layer="25"/>
-<circle x="53.975" y="14.605" radius="0.0635" width="0.4064" layer="25"/>
+<circle x="5.08" y="15.24" radius="0.0635" width="0.4064" layer="25"/>
+<circle x="19.685" y="15.24" radius="0.0635" width="0.4064" layer="25"/>
+<circle x="37.465" y="15.24" radius="0.0635" width="0.4064" layer="25"/>
+<circle x="47.625" y="15.24" radius="0.0635" width="0.4064" layer="25"/>
+<circle x="53.975" y="15.24" radius="0.0635" width="0.4064" layer="25"/>
 <text x="2.2225" y="5.08" size="1.016" layer="26" rot="MR90">GND</text>
 <text x="4.7625" y="5.08" size="1.016" layer="26" rot="MR90">Center</text>
@@
 <attribute name="VALUE" x="56.769" y="9.4615" size="1.27" layer="27" rot="R270"/>
 </element>
-<element name="C7" library="resistor" package="C0805" value="10pF" x="15.875" y="12.3825" smashed="yes">
+<element name="C7" library="resistor" package="C0805" value="5pF" x="15.875" y="12.3825" smashed="yes">
 <attribute name="NAME" x="18.669" y="11.4935" size="1.016" layer="25" rot="R90"/>
 <attribute name="VALUE" x="14.986" y="10.0965" size="1.27" layer="27"/>
@@
 <wire x1="40.005" y1="11.7475" x2="41.275" y2="11.7475" width="0.4064" layer="1"/>
 <wire x1="41.275" y1="11.7475" x2="42.545" y2="11.7475" width="0.4064" layer="1"/>
-<wire x1="61.595" y1="13.6525" x2="61.595" y2="13.5925" width="0" layer="19" extent="1-1"/>
+<wire x1="61.595" y1="13.5925" x2="61.595" y2="13.6525" width="0.3048" layer="1"/>
 </signal>
 <signal name="PW_CV">
