File: Xonik Waveshaper v2.2.brd (EAGLE design)
At the start: 55.9 x 21 mm, 99 parts, among them IC1 TL074JT, IC2 TL074JT, IC3 TL074JT, IC4 TL072JT, IC5 4013T, IC6 LM311T, T1 2n3904

Commit message: Switched to single connector
Parts:
- removed +12V, -12V, -2.5V, DCO_IN, GND, INV_SAW, IN_CENTER, PULSE, PULSE_AMP_CV, PW_CV, SAW, SINE, ST1, ST2, ST3, ST4, SUB_SAW_1, SUB_SAW_2, SUB_SQR_1, SUB_SQR_2, SYMMETRY, TRIANGLE: (no value), joakim:MA01N-1J
- added X1: (no value), joakim:MA22N-1J
Connections:
- net +12V: now also X1.20; no longer +12V.1
- net -12V: now also X1.22; no longer -12V.1
- net -5V: now also X1.11; no longer -2.5V.1
- net AMP_CV: now also X1.1; no longer PULSE_AMP_CV.1
- net DCO_IN: now also X1.4; no longer DCO_IN.1
- net GND: now also X1.21; no longer GND.1
- net INV_SAW: now also X1.8; no longer INV_SAW.1
- net IN_CENTER: now also X1.6; no longer IN_CENTER.1
- net PULSE: now also X1.3; no longer PULSE.1
- net PW_CV: now also X1.2; no longer PW_CV.1
- net SAW: now also X1.9; no longer SAW.1
- net SINE: now also X1.10; no longer SINE.1
- net SS1_TRIM_L: now also X1.16; no longer ST1.1
- net SS1_TRIM_R: now also X1.17; no longer ST2.1
- net SS2_TRIM_L: now also X1.14; no longer ST3.1
- net SS2_TRIM_R: now also X1.15; no longer ST4.1
- net SUB_SAW_1: now also X1.13; no longer SUB_SAW_1.1
- net SUB_SAW_2: now also X1.12; no longer SUB_SAW_2.1
- net SUB_SQR_1: now also X1.18; no longer SUB_SQR_1.1
- net SUB_SQR_2: now also X1.19; no longer SUB_SQR_2.1
- net SYMMETRY: now also X1.5; no longer SYMMETRY.1
- net TRIANGLE: now also X1.7; no longer TRIANGLE.1

Commit message: Updated footprints
Parts:
- C1, C14, C2, C3, C4, C5, C6, C7: device joakim:R0603-J -> joakim:C0603-J
- turned D1 to 90 degrees
- turned D2 to 90 degrees
- turned D3 to 270 degrees
- turned D4 to 90 degrees
Changed lines of the file:
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@@
 <attribute name="VALUE" x="21.11375" y="15.24" size="1.27" layer="27" rot="R270"/>
 </element>
-<element name="T1" library="transistor-neu-to92" package="SOT23-BEC" value="2n3904" x="1.905" y="17.145" smashed="yes" rot="R180">
+<element name="T1" library="transistor-neu-to92" library_urn="urn:adsk.eagle:library:397" package="SOT23-BEC" package3d_urn="urn:adsk.eagle:package:28748/2" value="2n3904" x="1.905" y="17.145" smashed="yes" rot="R180">
 <attribute name="NAME" x="1.27" y="19.20875" size="0.8128" layer="25" font="vector"/>
+<attribute name="POPULARITY" value="0" x="1.905" y="17.145" size="1.778" layer="27" rot="R180" display="off"/>
 <attribute name="VALUE" x="3.81" y="20.32" size="1.27" layer="27" rot="R180"/>
 </element>
@@
 <attribute name="VALUE" x="30.00375" y="6.0325" size="1.27" layer="27" rot="R270"/>
 </element>
-<element name="C1" library="joakim" package="R0603-J" value="10pF" x="41.11625" y="5.3975" smashed="yes" rot="R270">
+<element name="C1" library="joakim" package="C0603-J" value="10pF" x="41.11625" y="5.3975" smashed="yes" rot="R270">
 <attribute name="NAME" x="42.00525" y="3.8735" size="0.8128" layer="25" font="vector" rot="R180"/>
 <attribute name="VALUE" x="39.08425" y="6.2865" size="1.27" layer="27" rot="R270"/>
 </element>
-<element name="C2" library="joakim" package="R0603-J" value="10pF" x="39.84625" y="18.0975" smashed="yes" rot="R90">
+<element name="C2" library="joakim" package="C0603-J" value="10pF" x="39.84625" y="18.0975" smashed="yes" rot="R90">
 <attribute name="NAME" x="39.116" y="19.78025" size="0.8128" layer="25" font="vector"/>
 <attribute name="VALUE" x="41.87825" y="17.2085" size="1.27" layer="27" rot="R90"/>
 </element>
-<element name="C3" library="joakim" package="R0603-J" value="30pF" x="27.46375" y="14.605" smashed="yes" rot="R270">
+<element name="C3" library="joakim" package="C0603-J" value="30pF" x="27.46375" y="14.605" smashed="yes" rot="R270">
 <attribute name="NAME" x="26.7335" y="12.0015" size="0.8128" layer="25" font="vector"/>
 <attribute name="VALUE" x="25.43175" y="15.494" size="1.27" layer="27" rot="R270"/>
 </element>
-<element name="C4" library="joakim" package="R0603-J" value="30pF" x="27.46375" y="8.89" smashed="yes" rot="R90">
+<element name="C4" library="joakim" package="C0603-J" value="30pF" x="27.46375" y="8.89" smashed="yes" rot="R90">
 <attribute name="NAME" x="28.194" y="11.4935" size="0.8128" layer="25" font="vector" rot="R180"/>
 <attribute name="VALUE" x="29.49575" y="8.001" size="1.27" layer="27" rot="R90"/>
 </element>
-<element name="C5" library="joakim" package="R0603-J" value="100nF" x="52.86375" y="18.0975" smashed="yes" rot="R270">
+<element name="C5" library="joakim" package="C0603-J" value="100nF" x="52.86375" y="18.0975" smashed="yes" rot="R270">
 <attribute name="NAME" x="53.4035" y="19.78025" size="0.8128" layer="25" font="vector"/>
 <attribute name="VALUE" x="50.83175" y="18.9865" size="1.27" layer="27" rot="R270"/>
 </element>
-<element name="C6" library="joakim" package="R0603-J" value="100nF" x="54.45125" y="5.3975" smashed="yes" rot="R90">
+<element name="C6" library="joakim" package="C0603-J" value="100nF" x="54.45125" y="5.3975" smashed="yes" rot="R90">
 <attribute name="NAME" x="53.721" y="2.95275" size="0.8128" layer="25" font="vector"/>
 <attribute name="VALUE" x="56.48325" y="4.5085" size="1.27" layer="27" rot="R90"/>
 </element>
-<element name="C7" library="joakim" package="R0603-J" value="3pF" x="2.2225" y="9.525" smashed="yes" rot="R180">
+<element name="C7" library="joakim" package="C0603-J" value="3pF" x="2.2225" y="9.525" smashed="yes" rot="R180">
 <attribute name="NAME" x="3.1115" y="8.636" size="0.8128" layer="25" font="vector" rot="R180"/>
 <attribute name="VALUE" x="3.1115" y="11.557" size="1.27" layer="27" rot="R180"/>
@@
 <attribute name="VALUE" x="44.2" y="8.4975" size="1.27" layer="27" rot="R90"/>
 </element>
-<element name="D1" library="joakim" package="D0805-J" value="1N41480805" x="10.795" y="18.0975" smashed="yes" rot="R270">
+<element name="D1" library="joakim" package="D0805-J" value="1N41480805" x="10.795" y="18.0975" smashed="yes" rot="R90">
 <attribute name="NAME" x="10.19175" y="19.90725" size="0.8128" layer="25" font="vector"/>
-<attribute name="VALUE" x="8.509" y="18.8595" size="1.27" layer="27" rot="R270"/>
-</element>
-<element name="D2" library="joakim" package="D0805-J" value="1N41480805" x="13.0175" y="18.0975" smashed="yes" rot="R270">
+<attribute name="VALUE" x="13.081" y="17.3355" size="1.27" layer="27" rot="R90"/>
+</element>
+<element name="D2" library="joakim" package="D0805-J" value="1N41480805" x="13.0175" y="18.0975" smashed="yes" rot="R90">
 <attribute name="NAME" x="12.41425" y="19.90725" size="0.8128" layer="25" font="vector"/>
-<attribute name="VALUE" x="10.7315" y="18.8595" size="1.27" layer="27" rot="R270"/>
-</element>
-<element name="D3" library="joakim" package="D0805-J" value="1N41480805" x="23.01875" y="18.0975" smashed="yes" rot="R90">
-<attribute name="NAME" x="22.4155" y="19.90725" size="0.8128" layer="25" font="vector"/>
-<attribute name="VALUE" x="25.30475" y="17.3355" size="1.27" layer="27" rot="R90"/>
-</element>
-<element name="D4" library="joakim" package="D0805-J" value="1N41480805" x="25.24125" y="18.0975" smashed="yes" rot="R270">
-<attribute name="NAME" x="24.638" y="19.90725" size="0.8128" layer="25" font="vector"/>
-<attribute name="VALUE" x="22.95525" y="18.8595" size="1.27" layer="27" rot="R270"/>
+<attribute name="VALUE" x="15.3035" y="17.3355" size="1.27" layer="27" rot="R90"/>
+</element>
+<element name="D3" library="joakim" package="D0805-J" value="1N41480805" x="23.01875" y="18.0975" smashed="yes" rot="R270">
+<attribute name="NAME" x="22.4155" y="20.066" size="0.8128" layer="25" font="vector"/>
+<attribute name="VALUE" x="20.73275" y="18.8595" size="1.27" layer="27" rot="R270"/>
+</element>
+<element name="D4" library="joakim" package="D0805-J" value="1N41480805" x="25.24125" y="18.0975" smashed="yes" rot="R90">
+<attribute name="NAME" x="24.638" y="20.066" size="0.8128" layer="25" font="vector"/>
+<attribute name="VALUE" x="27.52725" y="17.3355" size="1.27" layer="27" rot="R90"/>
 </element>
 <element name="C16" library="joakim" package="C0402-J" value="1uF" x="33.655" y="6.82625" smashed="yes" rot="R90">
@@
 <attribute name="VALUE" x="48.645" y="8.4975" size="1.27" layer="27" rot="R90"/>
 </element>
-<element name="C14" library="joakim" package="R0603-J" value="820pF" x="46.51375" y="18.0975" smashed="yes" rot="R90">
+<element name="C14" library="joakim" package="C0603-J" value="820pF" x="46.51375" y="18.0975" smashed="yes" rot="R90">
 <attribute name="NAME" x="45.466" y="19.78025" size="0.8128" layer="25" font="vector"/>
 <attribute name="VALUE" x="48.54575" y="17.2085" size="1.27" layer="27" rot="R90"/>
@@
 <wire x1="8.89" y1="13.335" x2="9.525" y2="13.97" width="0.254" layer="1"/>
 <wire x1="9.525" y1="15.71625" x2="10.00125" y2="16.1925" width="0.254" layer="1"/>
-<wire x1="10.00125" y1="16.1925" x2="10.795" y2="16.1925" width="0.254" layer="1"/>
+<wire x1="10.00125" y1="16.1925" x2="10.4775" y2="16.1925" width="0.254" layer="1"/>
+<wire x1="10.4775" y1="16.1925" x2="10.795" y2="16.1925" width="0.254" layer="1"/>
 <wire x1="7.65" y1="13.78125" x2="8.09625" y2="13.335" width="0.254" layer="1"/>
 <wire x1="8.09625" y1="13.335" x2="8.89" y2="13.335" width="0.254" layer="1"/>
@@
 <contactref element="D2" pad="C"/>
 <contactref element="D1" pad="A"/>
-<wire x1="10.795" y1="19.0975" x2="11.85875" y2="19.0975" width="0.254" layer="1"/>
-<wire x1="11.85875" y1="19.0975" x2="12.065" y2="18.89125" width="0.254" layer="1"/>
-<wire x1="12.065" y1="18.89125" x2="12.065" y2="17.30375" width="0.254" layer="1"/>
-<wire x1="12.065" y1="17.30375" x2="12.27125" y2="17.0975" width="0.254" layer="1"/>
-<wire x1="12.27125" y1="17.0975" x2="13.0175" y2="17.0975" width="0.254" layer="1"/>
+<wire x1="10.795" y1="19.0975" x2="11.7" y2="19.0975" width="0.254" layer="1"/>
+<wire x1="11.7" y1="19.0975" x2="11.90625" y2="18.89125" width="0.254" layer="1"/>
+<wire x1="11.90625" y1="18.89125" x2="11.90625" y2="17.30375" width="0.254" layer="1"/>
+<wire x1="11.90625" y1="17.30375" x2="12.1125" y2="17.0975" width="0.254" layer="1"/>
+<wire x1="12.1125" y1="17.0975" x2="13.0175" y2="17.0975" width="0.254" layer="1"/>
 <wire x1="10.795" y1="19.0975" x2="10.04875" y2="19.0975" width="0.254" layer="1"/>
 <wire x1="10.04875" y1="19.0975" x2="9.525" y2="18.57375" width="0.254" layer="1"/>
@@
 <contactref element="15" pad="2"/>
 <contactref element="D2" pad="A"/>
-<wire x1="12.85875" y1="20.16125" x2="13.0175" y2="20.16125" width="0.254" layer="1"/>
 <wire x1="13.0175" y1="20.16125" x2="13.17625" y2="20.16125" width="0.254" layer="1"/>
-<wire x1="12.85875" y1="20.16125" x2="9.3425" y2="20.16125" width="0.254" layer="1"/>
+<wire x1="13.0175" y1="20.16125" x2="9.3425" y2="20.16125" width="0.254" layer="1"/>
 <wire x1="8.73125" y1="18.5975" x2="8.73125" y2="19.55" width="0.254" layer="1"/>
 <wire x1="9.3425" y1="20.16125" x2="8.73125" y2="19.55" width="0.254" layer="1"/>

Commit message: Checked with JLCPCB
Parts:
- moved X1 11.4 mm to (27.9, 1.27)
Changed lines of the file:
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@@
 <attribute name="VALUE" x="9.525" y="18.7325" size="1.27" layer="27" rot="R90"/>
 </element>
-<element name="X1" library="joakim" package="MA22N-1J" value="" x="16.51" y="1.27" smashed="yes">
-<attribute name="VALUE" x="54.61" y="-1.651" size="1.27" layer="27" ratio="10"/>
+<element name="X1" library="joakim" package="MA22N-1J" value="" x="27.94" y="1.27" smashed="yes">
+<attribute name="VALUE" x="66.04" y="-1.651" size="1.27" layer="27" ratio="10"/>
 </element>
 </elements>
@@
 <contactref element="5" pad="2"/>
 <wire x1="1.27" y1="4.5475" x2="1.27" y2="3.4925" width="0.254" layer="1"/>
+<wire x1="1.27" y1="3.4925" x2="1.27" y2="1.27" width="0.254" layer="1"/>
 <wire x1="1.27" y1="3.4925" x2="3.175" y2="3.4925" width="0.254" layer="1"/>
 <wire x1="3.4925" y1="3.81" x2="3.175" y2="3.4925" width="0.254" layer="1"/>
 <wire x1="3.4925" y1="3.81" x2="3.4925" y2="4.5475" width="0.254" layer="1"/>
-<wire x1="1.27" y1="1.27" x2="1.27" y2="3.4925" width="0.254" layer="1"/>
 <contactref element="X1" pad="1"/>
 </signal>
@@
 <wire x1="4.92125" y1="7.62" x2="4.92125" y2="6.50875" width="0.254" layer="16"/>
 <via x="4.92125" y="6.50875" extent="1-16" drill="0.3302"/>
+<wire x1="6.35" y1="1.42875" x2="5.08" y2="2.69875" width="0.254" layer="1"/>
+<wire x1="6.35" y1="1.42875" x2="6.35" y2="1.27" width="0.254" layer="1"/>
 <wire x1="4.92125" y1="6.50875" x2="5.08" y2="6.35" width="0.254" layer="1"/>
-<wire x1="5.08" y1="2.54" x2="6.35" y2="1.27" width="0.254" layer="1"/>
-<wire x1="5.08" y1="6.35" x2="5.08" y2="2.54" width="0.254" layer="1"/>
+<wire x1="5.08" y1="6.35" x2="5.08" y2="2.69875" width="0.254" layer="1"/>
 <wire x1="4.4" y1="8.9225" x2="4.4" y2="7.82375" width="0.254" layer="1"/>
 <wire x1="4.4" y1="7.82375" x2="4.445" y2="7.77875" width="0.254" layer="1"/>
@@
 <wire x1="18.57375" y1="4.28625" x2="13.97" y2="4.28625" width="0.254" layer="16"/>
 <via x="13.97" y="4.28625" extent="1-16" drill="0.3302"/>
-<wire x1="19.05" y1="1.27" x2="19.05" y2="3.01625" width="0.254" layer="1"/>
-<wire x1="19.05" y1="3.01625" x2="19.05" y2="3.4925" width="0.254" layer="1"/>
+<wire x1="19.05" y1="1.27" x2="19.05" y2="3.4925" width="0.254" layer="1"/>
 <wire x1="10.63625" y1="10.63625" x2="12.22375" y2="10.63625" width="0.254" layer="1"/>
 <wire x1="12.7" y1="8.09625" x2="13.096875" y2="7.699375" width="0.254" layer="1"/>
@@
 <via x="39.6875" y="3.6703" extent="1-16" drill="0.3302"/>
 <wire x1="39.6875" y1="3.6703" x2="40.65905" y2="2.69875" width="0.254" layer="16"/>
-<wire x1="43.02125" y1="2.69875" x2="44.45" y2="1.27" width="0.254" layer="16"/>
-<wire x1="40.65905" y1="2.69875" x2="43.02125" y2="2.69875" width="0.254" layer="16"/>
+<wire x1="43.03968125" y1="2.68031875" x2="43.03434375" y2="2.69875" width="0.254" layer="16"/>
+<wire x1="43.03968125" y1="2.68031875" x2="44.45" y2="1.27" width="0.254" layer="16"/>
+<wire x1="40.65905" y1="2.69875" x2="43.03434375" y2="2.69875" width="0.254" layer="16"/>
 <contactref element="X1" pad="18"/>
 </signal>
@@
 <wire x1="44.45" y1="3.65125" x2="44.45" y2="3.6703" width="0.254" layer="1"/>
 <via x="44.45" y="3.6703" extent="1-16" drill="0.3302"/>
-<wire x1="46.99" y1="1.27" x2="46.8503" y2="1.27" width="0.254" layer="16"/>
-<wire x1="46.8503" y1="1.27" x2="44.45" y2="3.6703" width="0.254" layer="16"/>
+<wire x1="46.99" y1="1.27" x2="46.961484375" y2="1.158815625" width="0.254" layer="16"/>
+<wire x1="46.961484375" y1="1.158815625" x2="44.45" y2="3.6703" width="0.254" layer="16"/>
 <contactref element="X1" pad="19"/>
 </signal>
@@
 <wire x1="30.7975" y1="13.35405" x2="30.7975" y2="13.755" width="0.254" layer="1"/>
 <via x="30.7975" y="4.28625" extent="1-16" drill="0.3302"/>
-<wire x1="30.7975" y1="2.2225" x2="31.75" y2="1.27" width="0.254" layer="16"/>
-<wire x1="30.7975" y1="4.28625" x2="30.7975" y2="2.2225" width="0.254" layer="16"/>
 <contactref element="X1" pad="13"/>
+<wire x1="31.75" y1="1.27" x2="30.7975" y2="2.2225" width="0.254" layer="16"/>
+<wire x1="30.7975" y1="2.2225" x2="30.7975" y2="4.28625" width="0.254" layer="16"/>
 </signal>
 <signal name="-5V">
@@
 <wire x1="47.78375" y1="3.65125" x2="47.78375" y2="4.5475" width="0.254" layer="1"/>
 <wire x1="47.78375" y1="3.65125" x2="46.83125" y2="2.69875" width="0.254" layer="1"/>
-<wire x1="26.67" y1="2.69875" x2="46.83125" y2="2.69875" width="0.254" layer="1"/>
 <wire x1="37.62375" y1="17.2475" x2="37.62375" y2="13.6525" width="0.254" layer="1"/>
 <wire x1="36.83" y1="12.85875" x2="34.29" y2="12.85875" width="0.254" layer="1"/>
@@
 <wire x1="37.62375" y1="13.6525" x2="36.83" y2="12.85875" width="0.254" layer="1"/>
 <wire x1="23.97125" y1="7.77875" x2="24.92375" y2="6.82625" width="0.254" layer="1"/>
-<wire x1="24.92375" y1="4.445" x2="26.67" y2="2.69875" width="0.254" layer="1"/>
-<wire x1="24.92375" y1="6.82625" x2="24.92375" y2="4.445" width="0.254" layer="1"/>
-<wire x1="26.67" y1="2.69875" x2="26.67" y2="1.27" width="0.254" layer="1"/>
+<wire x1="24.92375" y1="4.445" x2="24.92375" y2="6.82625" width="0.254" layer="1"/>
 <contactref element="X1" pad="11"/>
+<wire x1="26.67" y1="1.27" x2="26.67" y2="2.69875" width="0.254" layer="1"/>
+<wire x1="46.83125" y1="2.69875" x2="26.67" y2="2.69875" width="0.254" layer="1"/>
+<wire x1="26.67" y1="2.69875" x2="24.92375" y2="4.445" width="0.254" layer="1"/>
 </signal>
 <signal name="SS2_TRIM_R">
@@
 <wire x1="36.98875" y1="6.82625" x2="35.605" y2="8.21" width="0.254" layer="1"/>
 <via x="36.98875" y="3.81" extent="1-16" drill="0.3302"/>
-<wire x1="36.98875" y1="1.42875" x2="36.83" y2="1.27" width="0.254" layer="16"/>
-<wire x1="36.98875" y1="3.81" x2="36.98875" y2="1.42875" width="0.254" layer="16"/>
+<wire x1="36.98875" y1="1.310953125" x2="36.83" y2="1.27" width="0.254" layer="16"/>
+<wire x1="36.98875" y1="3.81" x2="36.98875" y2="1.310953125" width="0.254" layer="16"/>
 <contactref element="X1" pad="15"/>
 </signal>
@@
 <wire x1="26.035" y1="4.28625" x2="26.9875" y2="3.33375" width="0.254" layer="1"/>
 <via x="26.9875" y="3.33375" extent="1-16" drill="0.3302"/>
-<wire x1="29.21" y1="1.27" x2="29.05125" y2="1.27" width="0.254" layer="16"/>
-<wire x1="29.05125" y1="1.27" x2="26.9875" y2="3.33375" width="0.254" layer="16"/>
+<wire x1="29.21" y1="1.27" x2="29.1775875" y2="1.1436625" width="0.254" layer="16"/>
+<wire x1="29.1775875" y1="1.1436625" x2="26.9875" y2="3.33375" width="0.254" layer="16"/>
 <contactref element="X1" pad="12"/>
 </signal>
@@
 <wire x1="16.35125" y1="9.525" x2="16.35125" y2="2.38125" width="0.254" layer="1"/>
 <wire x1="16.35125" y1="2.38125" x2="16.35125" y2="2.2225" width="0.254" layer="1"/>
-<wire x1="16.35125" y1="2.38125" x2="16.35125" y2="1.42875" width="0.254" layer="1"/>
-<wire x1="16.35125" y1="1.42875" x2="16.51" y2="1.27" width="0.254" layer="1"/>
+<wire x1="16.35125" y1="2.38125" x2="16.35125" y2="1.311190625" width="0.254" layer="1"/>
+<wire x1="16.35125" y1="1.311190625" x2="16.51" y2="1.27" width="0.254" layer="1"/>
 <contactref element="X1" pad="7"/>
 </signal>
@@
 <wire x1="52.7177" y1="11.7348" x2="52.7177" y2="9.1948" width="0.508" layer="16"/>
 <via x="53.49875" y="2.8575" extent="1-16" drill="0.3302"/>
-<wire x1="53.49875" y1="2.8575" x2="51.1175" y2="2.8575" width="0.508" layer="1"/>
-<wire x1="51.1175" y1="2.8575" x2="49.53" y2="1.27" width="0.508" layer="1"/>
+<wire x1="53.49875" y1="2.8575" x2="50.95875" y2="2.8575" width="0.508" layer="1"/>
+<wire x1="50.95875" y1="2.8575" x2="49.53" y2="1.42875" width="0.508" layer="1"/>
+<wire x1="49.53" y1="1.42875" x2="49.53" y2="1.27" width="0.508" layer="1"/>
 <contactref element="X1" pad="20"/>
 </signal>
@@
 <via x="38.89375" y="4.3053" extent="1-16" drill="0.3302"/>
 <wire x1="39.21125" y1="9.8425" x2="39.21125" y2="4.60375" width="0.254" layer="1"/>
-<wire x1="41.29405" y1="1.27" x2="41.91" y2="1.27" width="0.254" layer="16"/>
-<wire x1="41.29405" y1="1.27" x2="38.89375" y2="3.6703" width="0.254" layer="16"/>
 <wire x1="38.89375" y1="4.3053" x2="38.89375" y2="3.6703" width="0.254" layer="16"/>
 <contactref element="X1" pad="17"/>
+<wire x1="38.89375" y1="3.6703" x2="41.29405" y2="1.27" width="0.254" layer="16"/>
+<wire x1="41.29405" y1="1.27" x2="41.91" y2="1.27" width="0.254" layer="16"/>
 </signal>
 <signal name="-12V">
@@
 <wire x1="55.245" y1="8.255" x2="53.6575" y2="9.8425" width="0.508" layer="16"/>
 <wire x1="55.245" y1="8.255" x2="55.245" y2="1.905" width="0.508" layer="16"/>
-<wire x1="55.245" y1="1.905" x2="54.61" y2="1.27" width="0.508" layer="16"/>
+<wire x1="54.61" y1="1.27" x2="55.245" y2="1.905" width="0.508" layer="16"/>
 <wire x1="43.4975" y1="9.86625" x2="43.4825" y2="10.00125" width="0.254" layer="1"/>
 <wire x1="43.4825" y1="10.00125" x2="42.70375" y2="10.00125" width="0.254" layer="1"/>
@@
 <wire x1="4.47773125" y1="5.99976875" x2="4.00148125" y2="6.47601875" width="0.254" layer="16"/>
 <via x="4.47773125" y="5.99976875" extent="1-16" drill="0.3302"/>
-<wire x1="4.47773125" y1="5.99976875" x2="4.47773125" y2="1.93773125" width="0.254" layer="1"/>
-<wire x1="4.47773125" y1="1.93773125" x2="3.81" y2="1.27" width="0.254" layer="1"/>
+<wire x1="4.47773125" y1="5.99976875" x2="4.47773125" y2="3.68398125" width="0.254" layer="1"/>
+<wire x1="3.81" y1="1.27" x2="3.81" y2="3.01625" width="0.254" layer="1"/>
+<wire x1="4.47773125" y1="3.68398125" x2="3.81" y2="3.01625" width="0.254" layer="1"/>
 <wire x1="4.00148125" y1="6.47601875" x2="4.00148125" y2="8.76398125" width="0.254" layer="16"/>
 <wire x1="4.00148125" y1="8.76398125" x2="5.3975" y2="10.16" width="0.254" layer="16"/>

Commit message: Changed to standard value on waveshaper comparator pullup
Parts:
- 1: value 500R -> 510R
Changed lines of the file:
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@@
 <attribute name="VALUE" x="48.54575" y="17.2085" size="1.27" layer="27" rot="R90"/>
 </element>
-<element name="1" library="rcl" library_urn="urn:adsk.eagle:library:334" package="R0603" package3d_urn="urn:adsk.eagle:package:23555/3" value="500R" x="48.73625" y="18.0975" smashed="yes" rot="R270">
+<element name="1" library="rcl" library_urn="urn:adsk.eagle:library:334" package="R0603" package3d_urn="urn:adsk.eagle:package:23555/3" value="510R" x="48.73625" y="18.0975" smashed="yes" rot="R270">
 <attribute name="NAME" x="48.5775" y="19.84375" size="0.8128" layer="25" font="vector"/>
 <attribute name="POPULARITY" value="70" x="48.73625" y="18.0975" size="1.778" layer="27" rot="R270" display="off"/>
